File: kicad/mg36kb.kicad_sch (KiCad schematic)
At the start: 90 parts, among them SW1 keyswitch, SW10 keyswitch, SW11 keyswitch, SW12 keyswitch, SW13 keyswitch, SW14 keyswitch, SW15 keyswitch, SW16 keyswitch, SW17 keyswitch, SW18 keyswitch, SW19 keyswitch, SW2 keyswitch, SW20 keyswitch, SW21 keyswitch, SW22 keyswitch, SW23 keyswitch, SW24 keyswitch, SW25 keyswitch, SW26 keyswitch, SW27 keyswitch, SW28 keyswitch, SW29 keyswitch, SW3 keyswitch, SW30 keyswitch, SW31 keyswitch, SW32 keyswitch, SW33 keyswitch, SW34 keyswitch, SW35 keyswitch, SW36 keyswitch, SW4 keyswitch, SW5 keyswitch, SW6 keyswitch, SW7 keyswitch, SW8 keyswitch, SW9 keyswitch, U1 Nice_Nano_V2, U2 Nice_Nano_V2

Commit message: init ergogen
Connections:
- net mosi2: now also U2.6 (3)
- net sck2: now also U2.5 (2)
Other:
- moved on the sheet: D16, D17, D21, D22, D23, D24, D25, D26, D27, D28, D29, D30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

Commit message: add logo img, continue schematic
Parts:
- added LSW1: SW_SPST, symbol Switch:SW_SPST
- added U3: SN74LV1T34DBV, Package_TO_SOT_SMD:SOT-23-5, symbol Logic_LevelTranslator:SN74LV1T34DBV
- added ksd1, ksd10, ksd11, ksd12, ksd13, ksd14, ksd15, ksd16, ksd17, ksd18, ksd2, ksd3, ksd4, ksd5, ksd6, ksd7, ksd8, ksd9: SK6803MINI-E, LED_SMD:LED_SK6812MINI_PLCC4_3.5x3.5mm_P1.75mm, symbol LED:SK6812MINI
- added led_con1_a, led_con1_a1, led_con1_b, led_con1_b1: Conn_01x03, symbol Connector_Generic:Conn_01x03
Connections:
- net +BATT1: now also LSW1.1 (A)
- net GND1: now also U3.3 (GND), ksd1.2 (VSS), ksd10.2 (VSS), ksd11.2 (VSS), ksd12.2 (VSS), ksd13.2 (VSS), ksd14.2 (VSS), ksd15.2 (VSS), ksd16.2 (VSS), ksd17.2 (VSS), ksd18.2 (VSS), ksd2.2 (VSS), ksd3.2 (VSS), ksd4.2 (VSS), ksd5.2 (VSS), ksd6.2 (VSS), ksd7.2 (VSS), ksd8.2 (VSS), ksd9.2 (VSS), led_con1_a.3 (Pin_3), led_con1_a1.3 (Pin_3), led_con1_b.3 (Pin_3), led_con1_b1.3 (Pin_3)
- net VCC1: now reaches Display1.3 (VCC)
- net VCC1: now also U1.21 (3.3v)
- net VCC2: now reaches Display2.3 (VCC)
- net VCC2: now also U2.21 (3.3v)
- net leds1: now reaches U1.2 (0)
- net leds1: now also U3.2 (A), U3.4 (Y), ksd1.3 (DIN), led_con1_a1.2 (Pin_2), led_con1_b1.2 (Pin_2)
- net leds2: now reaches U2.2 (0)
- new net: LSW1.2 (B), U3.5 (VCC), ksd1.4 (VDD), ksd10.4 (VDD), ksd11.4 (VDD), ksd12.4 (VDD), ksd13.4 (VDD), ksd14.4 (VDD), ksd15.4 (VDD), ksd16.4 (VDD), ksd17.4 (VDD), ksd18.4 (VDD), ksd2.4 (VDD), ksd3.4 (VDD), ksd4.4 (VDD), ksd5.4 (VDD), ksd6.4 (VDD), ksd7.4 (VDD), ksd8.4 (VDD), ksd9.4 (VDD), led_con1_a.1 (Pin_1), led_con1_a1.1 (Pin_1), led_con1_b.1 (Pin_1), led_con1_b1.1 (Pin_1)
- new net: ksd11.1 (DOUT), ksd12.3 (DIN)
- new net: ksd10.1 (DOUT), ksd11.3 (DIN)
- new net: ksd2.1 (DOUT), ksd3.3 (DIN)
- new net: ksd1.1 (DOUT), ksd2.3 (DIN)
- new net: ksd15.1 (DOUT), ksd16.3 (DIN), led_con1_a.2 (Pin_2), led_con1_b.2 (Pin_2)
- new net: ksd10.3 (DIN), ksd9.1 (DOUT)
- new net: ksd8.1 (DOUT), ksd9.3 (DIN)
- new net: ksd12.1 (DOUT), ksd13.3 (DIN)
- new net: ksd5.1 (DOUT), ksd6.3 (DIN)
- new net: ksd4.1 (DOUT), ksd5.3 (DIN)
- new net: ksd7.1 (DOUT), ksd8.3 (DIN)
- new net: ksd3.1 (DOUT), ksd4.3 (DIN)
- new net: ksd6.1 (DOUT), ksd7.3 (DIN)
- new net: ksd14.1 (DOUT), ksd15.3 (DIN)
- new net: ksd13.1 (DOUT), ksd14.3 (DIN)
- new net: ksd16.1 (DOUT), ksd17.3 (DIN)
- new net: ksd17.1 (DOUT), ksd18.3 (DIN)
- no-connect marks 0 -> 17
Other:
- moved on the sheet: Display1, rst1
